File: 3V_4I_ac_afe/kicad/3V_4I_ac_afe.kicad_pcb (KiCad board)
At the start: 2 copper layers, 140 x 60 mm, 116 parts, among them J1 screw, J10 screw, J11 V_ref, J12 VDDA, J13 SIGNAL, J14 GNDA, J15 AC L, J16 AC N, J17 screw, J18 V_ref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

Commit message: added few prototypes and script for zipping kicad gerbers
Parts:
- R12, R13, R23, R24, R34, R35: value R -> R_div_ref
- R14, R25, R36: value R -> 15K
