File: 3V_4I_ac_afe/kicad/ac_i_afe.sch (KiCad schematic (older format))
At the start: 13 parts, among them J1 screw, J2 CT_R, J3 CT_R, J4 V_ref, J5 VDDA, J6 SIGNAL, J7 GNDA, U1 MCP6021T

Commit message: added few prototypes and script for zipping kicad gerbers
Parts:
- C1: Description Kondensator: ceramiczny; MLCC; 4,7nF; 50V; X7R; ±10%; SMD; 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 -> (none); PART_ID 06035C472K4Z2A -> (none); PRODUCER AVX -> (none)
- R1: Description Rezystor: thin film; SMD; 0207 melf; 10Ω; 1W; ±1%; Ø2,2x5,8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 -> (none); PART_ID SMDMM0207-10R -> (none); PRODUCER VISHAY -> (none)
- R2: Description Rezystor: thick film; SMD; 0603; 1kΩ; 0,1W; ±1%; -55÷155°C -> (none); PART_ID 0603SAF1001T5E -> (none); PRODUCER ROYAL OHM -> (none)
- R3: Description Rezystor: thick film; SMD; 0603; 15kΩ; 0,1W; ±1%; -55÷155°C -> (none); PART_ID 0603SAF1502T5E -> (none); PRODUCER ROYAL OHM -> (none)
- U1: Description Wzmacniacz operacyjny; 10MHz; 2,5÷5,5V; Kanały: 1; SOT23-5 -> (none); PART_ID MCP6021T-E/OT -> (none); PRODUCER MICROCHIP -> (none)
Changed lines of the file:
@@
 $Descr A4 11693 8268
 encoding utf-8
-Sheet 6 8
+Sheet 2 8
 Title "Analog front end - pomiar prądu AC"
 Date "2020-11-06"
@@
 AR Path="/5FA5F6C5/5F427561" Ref="R40"  Part="1"
 AR Path="/5FA5FFA2/5F427561" Ref="R43"  Part="1"
-F 0 "R37" H 4720 4046 50  0000 L CNN
+F 0 "R1" H 4720 4046 50  0000 L CNN
 F 1 "10" H 4720 3955 50  0000 L CNN
 F 2 "Resistor_SMD:R_MELF_MMB-0207" V 4580 4000 50  0001 C CNN
 F 3 "https://www.tme.eu/pl/details/smdmm0207-10r/rezystory-smd-melf-0207/vishay/smm02070c1009fbp00/" H 4650 4000 50  0001 C CNN
-F 4 " SMM02070C1009FBP00" H 4650 4000 50  0001 C CNN "PART_ID"
-F 5 "VISHAY" H 4650 4000 50  0001 C CNN "PRODUCER"
-F 6 "SMDMM0207-10R" H 4650 4000 50  0001 C CNN "PART_ID"
-F 7 "Rezystor: thin film; SMD; 0207 melf; 10Ω; 1W; ±1%; Ø2,2x5,8mm" H 4650 4000 50  0001 C CNN "Description"
 	1    4650 4000
 	1    0    0    1
@@
 AR Path="/5FA5F6C5/5F427575" Ref="C3"  Part="1"
 AR Path="/5FA5FFA2/5F427575" Ref="C4"  Part="1"
-F 0 "C2" V 5850 3050 50  0000 C CNN
+F 0 "C1" V 5850 3050 50  0000 C CNN
 F 1 "4,7n" V 5950 3050 50  0000 C CNN
 F 2 "Capacitor_SMD:C_0603_1608Metric" H 6138 2900 50  0001 C CNN
 F 3 "https://www.tme.eu/pl/details/06035c472k4z2a/kondensatory-mlcc-smd-0603/avx/" H 6100 3050 50  0001 C CNN
-F 4 "AVX " H 6100 3050 50  0001 C CNN "PRODUCER"
-F 5 "Kondensator: ceramiczny; MLCC; 4,7nF; 50V; X7R; ±10%; SMD; 0603" H 6100 3050 50  0001 C CNN "Description"
-F 6 "06035C472K4Z2A" H 6100 3050 50  0001 C CNN "PART_ID"
 	1    6100 3050
 	0    1    1    0
@@
 AR Path="/5FA5F6C5/5F427585" Ref="R42"  Part="1"
 AR Path="/5FA5FFA2/5F427585" Ref="R45"  Part="1"
-F 0 "R39" V 5893 3450 50  0000 C CNN
+F 0 "R3" V 5893 3450 50  0000 C CNN
 F 1 "15K" V 5984 3450 50  0000 C CNN
 F 2 "Resistor_SMD:R_0603_1608Metric" V 6030 3450 50  0001 C CNN
 F 3 "https://www.tme.eu/pl/details/smd0603-15k-1%25/rezystory-smd-0603/royal-ohm/0603saf1502t5e/" H 6100 3450 50  0001 C CNN
-F 4 " 0603SAF1502T5E" H 6100 3450 50  0001 C CNN "PART_ID"
-F 5 "ROYAL OHM" H 6100 3450 50  0001 C CNN "PRODUCER"
-F 6 "0603SAF1502T5E" H 6100 3450 50  0001 C CNN "PART_ID"
-F 7 "Rezystor: thick film; SMD; 0603; 15kΩ; 0,1W; ±1%; -55÷155°C" H 6100 3450 50  0001 C CNN "Description"
 	1    6100 3450
 	0    1    1    0
@@
 AR Path="/5FA5F6C5/5F3FBA52" Ref="R41"  Part="1"
 AR Path="/5FA5FFA2/5F3FBA52" Ref="R44"  Part="1"
-F 0 "R38" V 4893 3450 50  0000 C CNN
+F 0 "R2" V 4893 3450 50  0000 C CNN
 F 1 "1K" V 4984 3450 50  0000 C CNN
 F 2 "Resistor_SMD:R_0603_1608Metric" V 5030 3450 50  0001 C CNN
 F 3 "https://www.tme.eu/pl/details/smd0603-1k-1%25/rezystory-smd-0603/royal-ohm/0603saf1001t5e/" H 5100 3450 50  0001 C CNN
-F 4 " 0603SAF1001T5E" H 5100 3450 50  0001 C CNN "PART_ID"
-F 5 "ROYAL OHM" H 5100 3450 50  0001 C CNN "PRODUCER"
-F 6 "0603SAF1001T5E" H 5100 3450 50  0001 C CNN "PART_ID"
-F 7 "Rezystor: thick film; SMD; 0603; 1kΩ; 0,1W; ±1%; -55÷155°C" H 5100 3450 50  0001 C CNN "Description"
 	1    5100 3450
 	0    1    1    0
@@
 AR Path="/5FA5F6C5/5F3FBA56" Ref="U6"  Part="1"
 AR Path="/5FA5FFA2/5F3FBA56" Ref="U7"  Part="1"
-F 0 "U5" H 6200 4400 50  0000 C CNN
+F 0 "U1" H 6200 4400 50  0000 C CNN
 F 1 "MCP6021T" H 6200 4300 50  0000 C CNN
 F 2 "Package_TO_SOT_SMD:SOT-23-5" H 5800 3950 50  0001 L CNN
 F 3 "https://www.tme.eu/pl/details/mcp6021t-e_ot/wzmacniacze-operacyjne-smd/microchip-technology/" H 5900 4350 50  0001 C CNN
-F 4 "Wzmacniacz operacyjny; 10MHz; 2,5÷5,5V; Kanały: 1; SOT23-5" H 5900 4150 50  0001 C CNN "Description"
-F 5 " MCP6021T-E/OT" H 5900 4150 50  0001 C CNN "PART_ID"
-F 6 "MICROCHIP" H 5900 4150 50  0001 C CNN "PRODUCER"
 	1    5900 4150
 	1    0    0    1
@@
 AR Path="/5FA5F6C5/5FA86B38" Ref="J39"  Part="1"
 AR Path="/5FA5FFA2/5FA86B38" Ref="J46"  Part="1"
-F 0 "J32" H 10430 3542 50  0000 L CNN
+F 0 "J4" H 10430 3542 50  0000 L CNN
 F 1 "V_ref" H 10430 3451 50  0000 L CNN
 F 2 "Connector_PinHeader_2.54mm:PinHeader_1x02_P2.54mm_Vertical" H 10350 3550 50  0001 C CNN
@@
 AR Path="/5FA5F6C5/5FA88690" Ref="J40"  Part="1"
 AR Path="/5FA5FFA2/5FA88690" Ref="J47"  Part="1"
-F 0 "J33" H 10430 3942 50  0000 L CNN
+F 0 "J5" H 10430 3942 50  0000 L CNN
 F 1 "VDDA" H 10430 3851 50  0000 L CNN
 F 2 "Connector_PinHeader_2.54mm:PinHeader_1x02_P2.54mm_Vertical" H 10350 3950 50  0001 C CNN
@@
 AR Path="/5FA5F6C5/5FA88B28" Ref="J41"  Part="1"
 AR Path="/5FA5FFA2/5FA88B28" Ref="J48"  Part="1"
-F 0 "J34" H 10430 4342 50  0000 L CNN
+F 0 "J6" H 10430 4342 50  0000 L CNN
 F 1 "SIGNAL" H 10430 4251 50  0000 L CNN
 F 2 "Connector_PinHeader_2.54mm:PinHeader_1x02_P2.54mm_Vertical" H 10350 4350 50  0001 C CNN
@@
 AR Path="/5FA5F6C5/5FA88D1D" Ref="J42"  Part="1"
 AR Path="/5FA5FFA2/5FA88D1D" Ref="J49"  Part="1"
-F 0 "J35" H 10430 4742 50  0000 L CNN
+F 0 "J7" H 10430 4742 50  0000 L CNN
 F 1 "GNDA" H 10430 4651 50  0000 L CNN
 F 2 "Connector_PinHeader_2.54mm:PinHeader_1x02_P2.54mm_Vertical" H 10350 4750 50  0001 C CNN
@@
 AR Path="/5FA5F6C5/5FA5EF6A" Ref="J37"  Part="1"
 AR Path="/5FA5FFA2/5FA5EF6A" Ref="J44"  Part="1"
-F 0 "J30" V 4900 3100 50  0000 C CNN
+F 0 "J2" V 4900 3100 50  0000 C CNN
 F 1 "CT_R" V 4800 3100 50  0000 C CNN
 F 2 "Connector_PinHeader_2.54mm:PinHeader_1x01_P2.54mm_Vertical" H 4650 3100 50  0001 C CNN
@@
 AR Path="/5FA5F6C5/5FA5FA9E" Ref="J38"  Part="1"
 AR Path="/5FA5FFA2/5FA5FA9E" Ref="J45"  Part="1"
-F 0 "J31" V 4900 4900 50  0000 C CNN
+F 0 "J3" V 4900 4900 50  0000 C CNN
 F 1 "CT_R" V 4800 4900 50  0000 C CNN
 F 2 "Connector_PinHeader_2.54mm:PinHeader_1x01_P2.54mm_Vertical" H 4650 4900 50  0001 C CNN
@@
 AR Path="/5FA5E85E/5FA6EE53" Ref="J?"  Part="1"
 AR Path="/5FA5EA5F/5FA6EE53" Ref="J?"  Part="1"
-F 0 "J29" H 1980 3942 50  0000 L CNN
+F 0 "J1" H 1980 3942 50  0000 L CNN
 F 1 "screw" H 1980 3851 50  0000 L CNN
 F 2 "TerminalBlock_Phoenix:TerminalBlock_Phoenix_PT-1,5-2-5.0-H_1x02_P5.00mm_Horizontal" H 1900 3950 50  0001 C CNN
@@
 AR Path="/5FA5F6C5/5FA7078B" Ref="CT3"  Part="1"
 AR Path="/5FA5FFA2/5FA7078B" Ref="CT4"  Part="1"
-F 0 "CT2" V 4100 5350 50  0000 R CNN
+F 0 "CT1" V 4100 5350 50  0000 R CNN
 F 1 "Current_Transformer" V 4100 5050 50  0000 R CNN
 F 2 "eMKa_TRAFO:CT_talema_pimary_wire" H 4100 3800 50  0001 C CNN
