File: stm32f373rct6_evaluation_board/kicad/stm32f373rct6_evaluation_board.kicad_pcb (KiCad board)
At the start: 2 copper layers, 100 x 50 mm, 79 parts, among them J1 RS485_connector, J2 Conn_02x03_Odd_Even, J3 Conn_01x08, J4 Conn_02x08_Odd_Even, J5 Conn_02x08_Odd_Even, J6 Conn_02x08_Odd_Even, J7 Conn_02x04_Odd_Even, SW1 SW, SW2 SW, SW3 SW_RESET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

Commit message: added few prototypes and script for zipping kicad gerbers
Parts:
- removed BT1: Battery_Cell, Battery:BatteryHolder_Keystone_2998_1x6.8mm
- removed D1, D2: STPS0530Z, Diode_SMD:D_SOD-123
Connections:
- U6 pad 1: +BATT -> VDD
Routing:
- net Net-(BT1-Pad1): track 63.9 -> 0.00 mm, vias 2 -> 0
- net +BATT: track 12.6 -> 0.00 mm
- net VDD: track 10.9 -> 14.6 mm
- net GND: vias 21 -> 18
