File: stm32f373rct6_evaluation_board/kicad/stm32f373rct6_evaluation_board.sch (KiCad schematic (older format))
At the start: 35 parts, among them J1 RS485_connector, J2 Conn_02x03_Odd_Even, J3 Conn_01x08, J4 Conn_02x08_Odd_Even, J5 Conn_02x08_Odd_Even, J6 Conn_02x08_Odd_Even, J7 Conn_02x04_Odd_Even, SW1 SW, SW2 SW, U1 AP2127K-3.3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

Commit message: added few prototypes and script for zipping kicad gerbers
Parts:
- removed BT1: Battery_Cell, Battery:BatteryHolder_Keystone_2998_1x6.8mm, symbol Device:Battery_Cell
- removed D1, D2: STPS0530Z, Diode_SMD:D_SOD-123, symbol Device:D_Schottky
Changed lines of the file:
@@
 $EndDescr
-$Comp
-L Device:Battery_Cell BT1
-U 1 1 5FCE5A36
-P 3950 950
-F 0 "BT1" V 3695 1000 50  0000 C CNN
-F 1 "Battery_Cell" V 3786 1000 50  0000 C CNN
-F 2 "Battery:BatteryHolder_Keystone_2998_1x6.8mm" V 3950 1010 50  0001 C CNN
-F 3 "~" V 3950 1010 50  0001 C CNN
-	1    3950 950
-	0    1    1    0
-$EndComp
-$Comp
-L Device:D_Schottky D1
-U 1 1 5FCFEA67
-P 4550 950
-F 0 "D1" H 4550 733 50  0000 C CNN
-F 1 " STPS0530Z" H 4550 824 50  0000 C CNN
-F 2 "Diode_SMD:D_SOD-123" H 4550 950 50  0001 C CNN
-F 3 "~" H 4550 950 50  0001 C CNN
-	1    4550 950
-	-1   0    0    1
-$EndComp
-Wire Wire Line
-	4400 950  4150 950
-$Comp
-L power:GND #PWR011
-U 1 1 5FD27247
-P 3400 950
-F 0 "#PWR011" H 3400 700 50  0001 C CNN
-F 1 "GND" V 3405 822 50  0000 R CNN
-F 2 "" H 3400 950 50  0001 C CNN
-F 3 "" H 3400 950 50  0001 C CNN
-	1    3400 950
-	0    1    -1   0
-$EndComp
-Wire Wire Line
-	3400 950  3850 950
-Wire Wire Line
-	4850 950  4700 950
-Wire Wire Line
-	4850 950  4850 1050
-Connection ~ 4850 1050
-Wire Wire Line
-	4850 1050 4850 1150
-Wire Wire Line
-	4700 1150 4850 1150
-Wire Wire Line
-	3400 1150 4400 1150
-$Comp
-L Device:D_Schottky D2
-U 1 1 5FD1992A
-P 4550 1150
-F 0 "D2" H 4550 1367 50  0000 C CNN
-F 1 " STPS0530Z" H 4550 1276 50  0000 C CNN
-F 2 "Diode_SMD:D_SOD-123" H 4550 1150 50  0001 C CNN
-F 3 "~" H 4550 1150 50  0001 C CNN
-	1    4550 1150
-	-1   0    0    1
-$EndComp
 $Comp
 L Connector_Generic:Conn_02x03_Odd_Even J2
@@
 L power:GND #PWR022
 U 1 1 5FED269B
-P 5250 3850
-F 0 "#PWR022" H 5250 3600 50  0001 C CNN
-F 1 "GND" V 5255 3722 50  0000 R CNN
-F 2 "" H 5250 3850 50  0001 C CNN
-F 3 "" H 5250 3850 50  0001 C CNN
-	1    5250 3850
+P 5250 3650
+F 0 "#PWR022" H 5250 3400 50  0001 C CNN
+F 1 "GND" V 5255 3522 50  0000 R CNN
+F 2 "" H 5250 3650 50  0001 C CNN
+F 3 "" H 5250 3650 50  0001 C CNN
+	1    5250 3650
 	0    -1   -1   0
 $EndComp
 Wire Wire Line
-	5250 3850 5000 3850
+	5250 3650 5000 3650
 Wire Wire Line
 	5000 3550 5250 3550
 $Sheet
-S 3650 3450 1350 500
+S 3650 3450 1350 800
 U 5FC81CFA
 F0 "ISOLATED RS485" 50
 F1 "sub_sch/isolated_rs485_transceiver.sch" 50
-F2 "GND_HOST" I R 5000 3850 50
+F2 "GND_HOST" I R 5000 3650 50
 F3 "VDD_BUS" I L 3650 3550 50
 F4 "RX_(out)" I R 5000 3750 50
@@
 F7 "RS485_A" I L 3650 3750 50
 F8 "VDD_HOST" I R 5000 3550 50
-F9 "TX_(in)" I R 5000 3650 50
+F9 "TX_(in)" I R 5000 3850 50
+F10 "DE" I R 5000 3950 50
+F11 "~RE" I R 5000 4050 50
 $EndSheet
 $Sheet
@@
 F18 "I2C_1_SDA" I L 7000 2900 50
 F19 "GPIO_PB5" I L 7000 3100 50
-F20 "USART3_RX_(in)" I L 7000 3750 50
-F21 "USART3_T_(out)" I L 7000 3650 50
+F20 "USART3_RX_(in)" I L 7000 3850 50
+F21 "USART3_T_(out)" I L 7000 3750 50
 F22 "VBAT" I L 7000 1050 50
 F23 "C6" I R 8800 2650 50
@@
 uC_SWD_CLK
 Wire Wire Line
-	7000 3650 5000 3650
-Wire Wire Line
-	5000 3750 7000 3750
+	7000 3750 5000 3750
+Wire Wire Line
+	5000 3850 7000 3850
 Wire Wire Line
 	7000 2900 5900 2900
@@
 	4700 1950 7000 1950
 Wire Wire Line
-	4850 1050 5500 1050
-$Comp
-L power:+BATT #PWR025
-U 1 1 60606EA1
-P 6000 950
-F 0 "#PWR025" H 6000 800 50  0001 C CNN
-F 1 "+BATT" H 6015 1123 50  0000 C CNN
-F 2 "" H 6000 950 50  0001 C CNN
-F 3 "" H 6000 950 50  0001 C CNN
-	1    6000 950
-	1    0    0    -1
-$EndComp
-Wire Wire Line
-	6000 950  6000 1050
-Connection ~ 6000 1050
-Wire Wire Line
-	6000 1050 7000 1050
+	6500 1050 7000 1050
 $Comp
 L power:VDD #PWR012
 U 1 1 6062D398
-P 3400 1150
-F 0 "#PWR012" H 3400 1000 50  0001 C CNN
-F 1 "VDD" V 3415 1277 50  0000 L CNN
-F 2 "" H 3400 1150 50  0001 C CNN
-F 3 "" H 3400 1150 50  0001 C CNN
-	1    3400 1150
+P 6500 1050
+F 0 "#PWR012" H 6500 900 50  0001 C CNN
+F 1 "VDD" V 6515 1177 50  0000 L CNN
+F 2 "" H 6500 1050 50  0001 C CNN
+F 3 "" H 6500 1050 50  0001 C CNN
+	1    6500 1050
 	0    -1   -1   0
 $EndComp
@@
 	1850 1100 1600 1100
 $Comp
-L power:PWR_FLAG #FLG03
-U 1 1 5FAE6781
-P 5500 950
-F 0 "#FLG03" H 5500 1025 50  0001 C CNN
-F 1 "PWR_FLAG" H 5500 1123 50  0000 C CNN
-F 2 "" H 5500 950 50  0001 C CNN
-F 3 "~" H 5500 950 50  0001 C CNN
-	1    5500 950
-	1    0    0    -1
-$EndComp
-Wire Wire Line
-	5500 950  5500 1050
-Connection ~ 5500 1050
-Wire Wire Line
-	5500 1050 6000 1050
-$Comp
 L Switch:SW_Push SW?
